File: NMEA-Sensorboard.brd (EAGLE design)
At the start: 56.7 x 48.9 mm, 15 parts, among them IC1 R-78E05-1.0, IC3 MCP2562, IC4 INA226, X3 DS1820, X4 DS1820, X5 DS1820, X6 DS1820, X7 BUS

Commit message: Sensor oun changed
Parts:
- renumbered I2 to IC2
Connections:
- net N$9: now also IC2.SVP; no longer IC2.IO18
Routing:
- net +3V3: track 122.6 -> 114.1 mm
- net N$9: track 59.8 -> 65.2 mm
Other:
- board text added: "+"
- board text added: "-"
- board text added: "NMEA-Sensorboard AZ 2023-06-11 v2"
Changed lines of the file:
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@@
 <layer number="43" name="vRestrict" color="2" fill="10" visible="yes" active="yes"/>
 <layer number="44" name="Drills" color="7" fill="1" visible="no" active="yes"/>
-<layer number="45" name="Holes" color="7" fill="1" visible="no" active="yes"/>
+<layer number="45" name="Holes" color="7" fill="1" visible="yes" active="yes"/>
 <layer number="46" name="Milling" color="3" fill="1" visible="no" active="yes"/>
 <layer number="47" name="Measures" color="7" fill="1" visible="yes" active="yes"/>
@@
 <text x="26.67" y="7.747" size="1.27" layer="25">H</text>
 <text x="31.75" y="7.747" size="1.27" layer="25">L</text>
+<text x="40.64" y="7.747" size="1.27" layer="25">+</text>
+<text x="45.72" y="7.747" size="1.27" layer="25">-</text>
+<text x="1.397" y="0.762" size="1.016" layer="25">NMEA-Sensorboard
+AZ 2023-06-11 v2</text>
+<rectangle x1="3.429" y1="21.59" x2="5.461" y2="41.91" layer="21"/>
+<rectangle x1="26.289" y1="21.59" x2="28.321" y2="41.91" layer="21"/>
 </plain>
 <attributes>
@@
 <elements>
 <element name="D1" library="_smd" package="SOD80" value="1N4001" x="43.434" y="12.573" smashed="yes" rot="R270">
-<attribute name="NAME" x="42.418" y="8.255" size="1.27" layer="25" ratio="10"/>
+<attribute name="NAME" x="42.545" y="15.494" size="1.27" layer="25" ratio="10"/>
 <attribute name="VALUE" x="40.64" y="14.605" size="1.27" layer="27" ratio="10" rot="R270"/>
 </element>
-<element name="I2" library="_esp32" package="ESP32_D1_MINI" value="ESP32_D1_MINI" x="29.845" y="17.78" smashed="yes" rot="R180">
-<attribute name="NAME" x="2.286" y="14.224" size="1.27" layer="25" rot="R180"/>
+<element name="IC2" library="_esp32" package="ESP32_D1_MINI" value="ESP32_D1_MINI" x="29.845" y="17.78" smashed="yes" rot="R180">
+<attribute name="NAME" x="1.016" y="14.224" size="1.27" layer="25" rot="R270"/>
 <attribute name="VALUE" x="19.685" y="10.16" size="1.27" layer="27" rot="R180"/>
 </element>
@@
 </element>
 <element name="IC3" library="_eigene" package="SO-8" value="MCP2562" x="16.3068" y="19.05" smashed="yes">
-<attribute name="NAME" x="17.526" y="23.0378" size="1.27" layer="25" ratio="10" rot="R180"/>
+<attribute name="NAME" x="17.526" y="15.9258" size="1.27" layer="25" ratio="10" rot="R180"/>
 <attribute name="VALUE" x="12.7508" y="18.415" size="1.27" layer="27" ratio="10"/>
 </element>
@@
 <signal name="RXD">
 <contactref element="IC3" pad="4"/>
-<contactref element="I2" pad="IO5"/>
+<contactref element="IC2" pad="IO5"/>
 <wire x1="12.6492" y1="17.2212" x2="13.5636" y2="17.2212" width="0.1524" layer="1"/>
 <wire x1="4.572" y1="25.2984" x2="12.6492" y2="17.2212" width="0.1524" layer="1"/>
@@
 <contactref element="X3" pad="3"/>
 <contactref element="IC4" pad="7"/>
-<contactref element="I2" pad="GND"/>
+<contactref element="IC2" pad="GND"/>
 <contactref element="X6" pad="3"/>
 <contactref element="X5" pad="3"/>
@@
 <wire x1="46.355" y1="35.56" x2="46.355" y2="42.926" width="0.8128" layer="16"/>
 <wire x1="46.355" y1="42.926" x2="46.609" y2="43.18" width="0.8128" layer="16"/>
-<contactref element="I2" pad="GND2"/>
+<contactref element="IC2" pad="GND2"/>
 <wire x1="21.59" y1="31.75" x2="24.13" y2="29.21" width="0.8128" layer="1"/>
 <wire x1="24.13" y1="29.21" x2="24.13" y2="27.94" width="0.8128" layer="1"/>
@@
 <contactref element="X3" pad="1"/>
 <contactref element="IC4" pad="8"/>
-<contactref element="I2" pad="3V3"/>
+<contactref element="IC2" pad="3V3"/>
 <contactref element="R1" pad="1"/>
 <contactref element="X6" pad="1"/>
@@
 <wire x1="8.255" y1="19.05" x2="8.255" y2="15.24" width="0.8128" layer="16"/>
 <wire x1="8.255" y1="15.24" x2="10.795" y2="12.7" width="0.8128" layer="16"/>
-<wire x1="34.925" y1="20.32" x2="34.925" y2="24.13" width="0.8128" layer="1"/>
-<wire x1="34.925" y1="24.13" x2="34.925" y2="27.94" width="0.8128" layer="1"/>
-<wire x1="34.925" y1="27.94" x2="34.925" y2="35.56" width="0.8128" layer="1"/>
+<wire x1="34.925" y1="20.32" x2="34.925" y2="27.94" width="0.8128" layer="1"/>
+<wire x1="34.925" y1="27.94" x2="34.925" y2="33.02" width="0.8128" layer="1"/>
+<wire x1="34.925" y1="33.02" x2="34.925" y2="35.56" width="0.8128" layer="1"/>
 <wire x1="34.925" y1="35.56" x2="34.925" y2="45.72" width="0.8128" layer="1"/>
 <contactref element="X7" pad="1"/>
-<wire x1="34.925" y1="24.13" x2="41.275" y2="24.13" width="0.8128" layer="1"/>
-<wire x1="41.275" y1="24.13" x2="43.815" y2="26.67" width="0.8128" layer="1"/>
-<wire x1="43.815" y1="26.67" x2="43.815" y2="35.56" width="0.8128" layer="1"/>
 <wire x1="10.795" y1="12.7" x2="34.925" y2="12.7" width="0.8128" layer="16"/>
 <wire x1="34.925" y1="12.7" x2="34.925" y2="20.32" width="0.8128" layer="16"/>
@@
 <wire x1="27.94" y1="12.7" x2="19.685" y2="20.955" width="0.1524" layer="1"/>
 <wire x1="19.685" y1="20.955" x2="19.05" y2="20.955" width="0.1524" layer="1"/>
+<wire x1="34.925" y1="33.02" x2="41.91" y2="33.02" width="0.8128" layer="1"/>
+<wire x1="41.91" y1="33.02" x2="43.815" y2="34.925" width="0.8128" layer="1"/>
+<wire x1="43.815" y1="34.925" x2="43.815" y2="35.56" width="0.8128" layer="1"/>
 </signal>
 <signal name="LOAD">
@@
 </signal>
 <signal name="SCL">
-<contactref element="I2" pad="IO22"/>
+<contactref element="IC2" pad="IO22"/>
 <contactref element="IC4" pad="6"/>
 <via x="37.465" y="40.64" extent="1-16" drill="0.35"/>
@@
 </signal>
 <signal name="SDA">
-<contactref element="I2" pad="IO21"/>
+<contactref element="IC2" pad="IO21"/>
 <contactref element="IC4" pad="5"/>
 <via x="36.195" y="39.878" extent="1-16" drill="0.35"/>
@@
 <signal name="ALE">
 <contactref element="IC4" pad="4"/>
-<contactref element="I2" pad="IO19"/>
+<contactref element="IC2" pad="IO19"/>
 <wire x1="43.815" y1="46.99" x2="45.085" y2="45.72" width="0.1524" layer="16"/>
 <wire x1="4.445" y1="30.48" x2="8.255" y2="34.29" width="0.1524" layer="16"/>
@@
 </signal>
 <signal name="N$9">
-<contactref element="I2" pad="IO18"/>
 <contactref element="R1" pad="2"/>
 <contactref element="X3" pad="2"/>
@@
 <contactref element="X5" pad="2"/>
 <contactref element="X4" pad="2"/>
-<wire x1="4.445" y1="33.02" x2="6.985" y2="33.02" width="0.1524" layer="1"/>
-<wire x1="6.985" y1="33.02" x2="10.795" y2="29.21" width="0.1524" layer="1"/>
-<wire x1="37.465" y1="35.56" x2="37.465" y2="27.94" width="0.1524" layer="1"/>
+<wire x1="37.465" y1="35.56" x2="37.465" y2="27.94" width="0.1524" layer="16"/>
 <wire x1="37.465" y1="20.32" x2="37.465" y2="12.7" width="0.1524" layer="16"/>
 <wire x1="10.795" y1="29.21" x2="13.335" y2="29.21" width="0.1524" layer="1"/>
@@
 <wire x1="13.335" y1="29.21" x2="32.385" y2="29.21" width="0.1524" layer="16"/>
 <wire x1="37.465" y1="20.32" x2="37.465" y2="27.94" width="0.1524" layer="16"/>
+<contactref element="IC2" pad="SVP"/>
+<wire x1="10.795" y1="29.21" x2="10.795" y2="34.925" width="0.1524" layer="1"/>
+<wire x1="10.795" y1="34.925" x2="7.62" y2="38.1" width="0.1524" layer="1"/>
+<wire x1="7.62" y1="38.1" x2="4.445" y2="38.1" width="0.1524" layer="1"/>
 </signal>
 <signal name="+5V">
-<contactref element="I2" pad="VCC"/>
+<contactref element="IC2" pad="VCC"/>
 <contactref element="IC1" pad="OUT"/>
 <wire x1="27.2542" y1="22.8092" x2="27.305" y2="22.86" width="0.1524" layer="1"/>
@@
 <signal name="TXD">
 <contactref element="IC3" pad="1"/>
-<contactref element="I2" pad="IO23"/>
+<contactref element="IC2" pad="IO23"/>
 <wire x1="11.43" y1="21.0312" x2="13.5636" y2="21.0312" width="0.1524" layer="1"/>
 <wire x1="4.572" y1="27.8892" x2="11.43" y2="21.0312" width="0.1524" layer="1"/>
@@
 </drawing>
 <compatibility>
+<note version="6.3" minversion="6.2.2" severity="warning">
+Since Version 6.2.2 text objects can contain more than one line,
+which will not be processed correctly with this version.
+</note>
 <note version="8.2" severity="warning">
 Since Version 8.2, EAGLE supports online libraries. The ids
