File: NMEA-Sensorboard.brd (EAGLE design)
At the start: 56.7 x 48.9 mm, 15 parts, among them IC1 R-78E05-1.0, IC2 ESP32_D1_MINI, IC3 MCP2562, IC4 INA226, X3 DS1820, X4 DS1820, X5 DS1820, X6 DS1820, X7 BUS

Commit message: refactor: overhaul schematic and PCB layout to fix multiple issues
Parts:
- C1: device rcl:E5-8,5 -> rcl:E2-5
- moved C1 1.27 mm to (49.3, 12.8)
Connections:
- net N$9 renamed DATA
- net +3V3: now also IC3.5; no longer IC3.8
- net CANH: now also IC3.7, X2.2; no longer IC3.6, X2.1
- net CANL: now also IC3.6, X2.1; no longer IC3.7, X2.2
- net GND: now also IC3.8; no longer IC3.5
- net RXD: now also IC2.IO17; no longer IC2.IO5
- net TXD: now also IC2.IO16; no longer IC2.IO23
Routing:
- net RXD: track 12.6 -> 27.9 mm
- net TXD: track 12.0 -> 23.0 mm
- net GND: track 150.2 -> 141.6 mm
- net +3V3: track 114.1 -> 105.5 mm
- net CANL: track 21.9 -> 18.5 mm
- net CANH: track 18.6 -> 21.9 mm
- net +5V: track 57.1 -> 58.8 mm
- net 12V: track 53.9 -> 55.3 mm
Other:
- board text added: "+12V"
- board text added: "+3.3V"
- board text added: "+5V"
- board text added: "ALE"
- board text added: "CS"
- board text added: "DATA"
- board text added: "GND"
- board text added: "IO26"
- board text added: "IO36"
- board text added: "Load"
- board text added: "MISO"
- board text added: "MOSI"
- board text added: "N2k-RXD"
- board text added: "N2k-TXD"
- board text added: "NMEA-Sensorboard AZ 2026-08-09 v3"
- board text added: "RST"
- board text added: "RXD"
- board text added: "SCK"
- board text added: "SCL"
- board text added: "SDA"
- board text added: "TXD"
- board text removed: "NMEA-Sensorboard AZ 2023-06-11 v2"
